Commit message: Update

File: dev_ws/src/diff_robot_description/urdf/control/ros2_controllers.xacro (robot description, xacro)
@@ -1,5 +1,5 @@
 <?xml version="1.0"?>
-<robot name="my_robot" xmlns:xacro="http://www.ros.org/wiki/xacro">
-    <ros2_control name="MobileRobotHWInterface" type="system">
+<robot name="my_diff_robot" xmlns:xacro="http://www.ros.org/wiki/xacro">
+    <ros2_control name="DiffMobileRobotHWInterface" type="system">
         <hardware>
             <plugin>mock_components/GenericSystem</plugin>

File: dev_ws/src/diff_robot_description/urdf/robot/mobile_base.xacro (robot description, xacro)
@@ -6,5 +6,20 @@
     <xacro:property name="wheel_radius" value="0.1" />
     <xacro:property name="wheel_length" value="0.05" />
+    <xacro:arg name="enable_collision" default="false" />
+    <xacro:macro name="default_inertia" params="mass">
+        <inertial>
+            <mass value="${mass}"/>
+            <origin xyz="0.0 0.0 0.0" rpy="0.0 0.0 0.0"/>
+            <inertia ixx="1" ixy="0.0" ixz="0.0" iyy="1" iyz="0.0" izz="1"/>
+        </inertial>
+    </xacro:macro>
+    <!-- base_footprint (projection of base_link on the ground) -->
     <link name="base_footprint" />
+    <joint name="base_joint" type="fixed">
+        <parent link="base_footprint" />
+        <child link="base_link" />
+        <origin xyz="0 0 ${wheel_radius}" rpy="0 0 0"/>
+    </joint>
+    <!-- base_link and base_scan (required for Nav2) -->
     <link name="base_link">
         <visual>
@@ -15,5 +30,14 @@
             <material name="blue" />
         </visual>
+    <xacro:if value="$(arg enable_collision)">
+        <collision>
+          <geometry>
+            <box size="${base_length} ${base_width} ${base_height}" />
+          </geometry>
+        </collision>
+      </xacro:if>
+      <xacro:default_inertia mass="1"/>
     </link>
+    <!-- 2 Differential wheels and one caster wheel to keep balance-->
     <xacro:macro name="wheel_link" params="prefix">
         <link name="${prefix}_wheel_link">
@@ -25,5 +49,13 @@
                 <material name="grey" />
             </visual>
-        </link>
+    <xacro:if value="$(arg enable_collision)">
+        <collision>
+          <geometry>
+            <cylinder radius="${wheel_radius}" length="${wheel_length}" />
+          </geometry>
+        </collision>
+      </xacro:if>
+      <xacro:default_inertia mass="1"/>
+    </link>
     </xacro:macro>
     <xacro:wheel_link prefix="right" />
@@ -37,10 +69,13 @@
             <material name="grey" />
         </visual>
+    <xacro:if value="$(arg enable_collision)">
+        <collision>
+          <geometry>
+            <sphere radius="${wheel_radius / 2.0}" />
+          </geometry>
+        </collision>
+      </xacro:if>
+      <xacro:default_inertia mass="1"/>
     </link>
-    <joint name="base_joint" type="fixed">
-        <parent link="base_footprint" />
-        <child link="base_link" />
-        <origin xyz="0 0 ${wheel_radius}" rpy="0 0 0"/>
-    </joint>
     <joint name="base_right_wheel_joint" type="continuous">
         <parent link="base_link" />

Commit message: adding nav2 nav

File: dev_ws/src/diff_robot_description/urdf/control/ros2_controllers.xacro (robot description, xacro)
@@ -1,9 +1,16 @@
 <?xml version="1.0"?>
 <robot name="my_diff_robot" xmlns:xacro="http://www.ros.org/wiki/xacro">
+    <xacro:arg name="enable_gz_control" default="false"/>
     <ros2_control name="DiffMobileRobotHWInterface" type="system">
         <hardware>
-            <plugin>mock_components/GenericSystem</plugin>
+            <xacro:if value="$(arg enable_gz_control)">
+                <plugin>gz_ros2_control/GazeboSimSystem</plugin>
+            </xacro:if>
+            <xacro:unless value="$(arg enable_gz_control)">
+                <plugin>mock_components/GenericSystem</plugin>
+            </xacro:unless>
             <param name="calculate_dynamics" >true</param>
         </hardware>
+        <!-- Command and State interfaces -->
         <joint name="base_right_wheel_joint">
             <command_interface name="velocity"/>

File: dev_ws/src/diff_robot_description/urdf/gazebo/gazebo.xacro (robot description, xacro)
@@ -4,13 +4,36 @@
     <xacro:property name="M_PI" value="3.1415926535897931" />
     <xacro:arg name="enable_collision" default="false"/>
+    <xacro:arg name="enable_gz_control" default="false"/>
     <xacro:include filename="$(find diff_robot_description)/urdf/sensors/imu.urdf.xacro" />
     <xacro:include filename="$(find diff_robot_description)/urdf/sensors/lidar.urdf.xacro" />
     <xacro:include filename="$(find diff_robot_description)/urdf/sensors/rgbd_camera.urdf.xacro" />
-<!--
+    <!-- Wheel properties-->
+    <gazebo reference="left_wheel_link">
+      <mu1>1</mu1>
+      <mu2>1</mu2>
+    </gazebo>
+    <gazebo reference="right_wheel_link">
+      <mu1>1</mu1>
+      <mu2>1</mu2>
+    </gazebo>
+    <gazebo reference="caster_wheel_link">
+      <mu1>0.01</mu1>
+      <mu2>0.01</mu2>
+    </gazebo>
+    <!-- Plugin Ros2 control Section for Gazebo-->
+    <xacro:if value="$(arg enable_gz_control)">
+      <gazebo>
+        <plugin filename="gz_ros2_control-system" name="gz_ros2_control::GazeboSimROS2ControlPlugin">
+            <parameters>$(find diff_robot_controllers)/config/robot_controllers.yaml</parameters>
+        </plugin>
+      </gazebo>
+    </xacro:if>
+    <!-- Sensors section -->
     <xacro:rgbd_camera
       prefix="$(arg prefix)"
       camera_name="cam_1"
-      xyz_offset="0.105 0 0.05"
-      rpy_offset="0 -0.50 0"/>
+      xyz_offset="0.3 0 0.1"
+      rpy_offset="0 0 0"
+      enable_collision="$(arg enable_collision)"/>
     <xacro:imu_sensor
       prefix="$(arg prefix)"
@@ -20,12 +43,13 @@
       rpy_offset="0 0 0"
       update_rate="15.0"
-      topic_name="imu/data"/> -->
-      <xacro:lidar_sensor
-        prefix="$(arg prefix)"
-        parent="base_link"
-        frame_id="base_scan"
-        xyz_offset="0 0 0.23"
-        rpy_offset="0 0 0"
-        enable_collision="$(arg enable_collision)"
-        topic_name="scan"/>
+      topic_name="imu/data"
+      enable_collision="$(arg enable_collision)"/>
+    <xacro:lidar_sensor
+      prefix="$(arg prefix)"
+      parent="base_link"
+      frame_id="base_scan"
+      xyz_offset="0 0 0.23"
+      rpy_offset="0 0 0"
+      enable_collision="$(arg enable_collision)"
+      topic_name="scan"/>
 </robot>

File: dev_ws/src/diff_robot_description/urdf/robot/common_properties.xacro (robot description, xacro)
@@ -7,3 +7,6 @@
         <color rgba="0.5 0.5 0.5 1" />
     </material>
+    <material name="black">
+        <color rgba="0 0 0 1" />
+    </material>
 </robot>

File: dev_ws/src/diff_robot_description/urdf/robot/mobile_base.xacro (robot description, xacro)
@@ -1,4 +1,5 @@
 <?xml version="1.0"?>
 <robot xmlns:xacro="http://www.ros.org/wiki/xacro">
+  <xacro:include filename="$(find diff_robot_description)/urdf/inertia.xacro" />
     <xacro:property name="base_length" value="0.6" />
     <xacro:property name="base_width" value="0.4" />
@@ -35,7 +36,10 @@
             <box size="${base_length} ${base_width} ${base_height}" />
           </geometry>
+          <origin xyz="0 0 ${base_height / 2.0}" rpy="0 0 0" />
         </collision>
       </xacro:if>
-      <xacro:default_inertia mass="1"/>
+      <xacro:inertial_box mass="5"  x="${base_length}" y="${base_width}" z="${base_height}">
+        <origin xyz="0 0 ${base_height / 2.0}" rpy="0 0 0"/>
+      </xacro:inertial_box>
     </link>
     <!-- 2 Differential wheels and one caster wheel to keep balance-->
@@ -44,18 +48,21 @@
             <visual>
                 <geometry>
-                    <cylinder radius="${wheel_radius}" length="${wheel_length}" />
+                    <cylinder radius="${wheel_radius}" length="${wheel_length}"/>
                 </geometry>
                 <origin xyz="0 0 0" rpy="${pi / 2.0} 0 0" />
-                <material name="grey" />
+                <material name="black" />
             </visual>
-    <xacro:if value="$(arg enable_collision)">
-        <collision>
-          <geometry>
-            <cylinder radius="${wheel_radius}" length="${wheel_length}" />
-          </geometry>
-        </collision>
-      </xacro:if>
-      <xacro:default_inertia mass="1"/>
-    </link>
+            <xacro:if value="$(arg enable_collision)">
+                <collision>
+                  <geometry>
+                    <cylinder radius="${wheel_radius}" length="${wheel_length}" />
+                  </geometry>
+                  <origin xyz="0 0 0" rpy="${pi / 2.0} 0 0" />
+                </collision>
+              </xacro:if>
+              <xacro:inertial_cylinder mass="1" length="${wheel_length}" radius="${wheel_radius}">
+                <origin xyz="0 0 0" rpy="${pi / 2.0} 0 0" />
+              </xacro:inertial_cylinder>
+          </link>
     </xacro:macro>
     <xacro:wheel_link prefix="right" />
@@ -67,14 +74,17 @@
             </geometry>
             <origin xyz="0 0 0" rpy="0 0 0" />
-            <material name="grey" />
+            <material name="black" />
         </visual>
-    <xacro:if value="$(arg enable_collision)">
-        <collision>
-          <geometry>
-            <sphere radius="${wheel_radius / 2.0}" />
-          </geometry>
-        </collision>
-      </xacro:if>
-      <xacro:default_inertia mass="1"/>
+        <xacro:if value="$(arg enable_collision)">
+            <collision>
+              <geometry>
+                <sphere radius="${wheel_radius / 2.0}" />
+              </geometry>
+              <origin xyz="0 0 0" rpy="0 0 0" />
+            </collision>
+        </xacro:if>
+        <xacro:inertial_sphere mass="0.5" radius="${wheel_radius / 2.0}">
+          <origin xyz="0 0 0" rpy="0 0 0" />
+        </xacro:inertial_sphere>
     </link>
     <joint name="base_right_wheel_joint" type="continuous">
@@ -83,4 +93,5 @@
         <origin xyz="${-base_length / 4.0} ${-(base_width + wheel_length) / 2.0} 0" rpy="0 0 0" />
         <axis xyz="0 1 0" />
+        <dynamics damping="0.1" friction="0.0"/>
     </joint>
     <joint name="base_left_wheel_joint" type="continuous">
@@ -89,4 +100,5 @@
         <origin xyz="${-base_length / 4.0} ${(base_width + wheel_length) / 2.0} 0" rpy="0 0 0" />
         <axis xyz="0 1 0" />
+        <dynamics damping="0.1" friction="0.0"/>
     </joint>
     <joint name="base_caster_wheel_joint" type="fixed">
@@ -94,4 +106,5 @@
         <child link="caster_wheel_link" />
         <origin xyz="${base_length / 3.0} 0 ${-wheel_radius / 2.0}" rpy="0 0 0" />
+        <axis xyz="0 0 1" />
     </joint>
 </robot>

File: dev_ws/src/diff_robot_description/urdf/robot/my_robot.urdf.xacro (robot description, xacro)
@@ -3,5 +3,5 @@
     <xacro:include filename="$(find diff_robot_description)/urdf/robot/common_properties.xacro" />
     <xacro:include filename="$(find diff_robot_description)/urdf/robot/mobile_base.xacro" />
+    <xacro:include filename="$(find diff_robot_description)/urdf/gazebo/gazebo.xacro" />
     <xacro:include filename="$(find diff_robot_description)/urdf/control/ros2_controllers.xacro" />
-    <xacro:include filename="$(find diff_robot_description)/urdf/gazebo/gazebo.xacro" />
 </robot>

File: dev_ws/src/diff_robot_description/urdf/sensors/imu.urdf.xacro (robot description, xacro)
@@ -22,5 +22,6 @@
         topic_name:='imu/data'
         always_on:=true
-        visualize:=false">
+        visualize:=false
+        enable_collision:=false">
         <xacro:property name="ixx" value="${(mass/12.0) * (height*height + width*width)}" />
         <xacro:property name="iyy" value="${(mass/12.0) * (length*length + height*height)}" />
@@ -47,4 +48,12 @@
                     izz="${izz}" />
             </inertial>
+            <xacro:if value="${enable_collision}">
+                <collision>
+                <geometry>
+                    <box size="${length} ${width} ${height}"/>
+                </geometry>
+                <origin xyz="${inertial_xyz_offset}" rpy="${inertial_rpy_offset}"/>s
+                </collision>
+            </xacro:if>
         </link>
         <joint name="${prefix}${frame_id}_joint" type="fixed">
@@ -53,4 +62,10 @@
             <origin xyz="${xyz_offset}" rpy="${rpy_offset}"/>
         </joint>
+        <!-- IMU Sensor -->
+        <gazebo>
+            <plugin filename="gz-sim-imu-system"
+                    name="gz::sim::systems::Imu">
+            </plugin>
+        </gazebo>
         <gazebo reference="${prefix}${frame_id}_link">
             <material>
@@ -65,4 +80,81 @@
                 <visualize>${visualize}</visualize>
                 <gz_frame_id>${prefix}${frame_id}_link</gz_frame_id>
+                <imu>
+                    <angular_velocity>true</angular_velocity>
+                    <linear_acceleration>true</linear_acceleration>
+                  </imu>
+                <!--<imu>
+                    <enable_orientation>0</enable_orientation>
+                    <angular_velocity>
+                      <x>
+                        <noise type="gaussian">
+                          <mean>0</mean>
+                          <stddev>0.009</stddev>
+                          <bias_mean>0.00075</bias_mean>
+                          <bias_stddev>0.005</bias_stddev>
+                          <dynamic_bias_stddev>0.00002</dynamic_bias_stddev>
+                          <dynamic_bias_correlation_time>400.0</dynamic_bias_correlation_time>
+                          <precision>0.00025</precision>
+                        </noise>
+                      </x>
+                      <y>
+                        <noise type="gaussian">
+                          <mean>0</mean>
+                          <stddev>0.009</stddev>
+                          <bias_mean>0.00075</bias_mean>
+                          <bias_stddev>0.005</bias_stddev>
+                          <dynamic_bias_stddev>0.00002</dynamic_bias_stddev>
+                          <dynamic_bias_correlation_time>400.0</dynamic_bias_correlation_time>
+                          <precision>0.00025</precision>
+                        </noise>
+                      </y>
+                      <z>
+                        <noise type="gaussian">
+                          <mean>0</mean>
+                          <stddev>0.009</stddev>
+                          <bias_mean>0.00075</bias_mean>
+                          <bias_stddev>0.005</bias_stddev>
+                          <dynamic_bias_stddev>0.00002</dynamic_bias_stddev>
+                          <dynamic_bias_correlation_time>400.0</dynamic_bias_correlation_time>
+                          <precision>0.00025</precision>
+                        </noise>
+                      </z>
+                    </angular_velocity>
+                    <linear_acceleration>
+                      <x>
+                        <noise type="gaussian">
+                          <mean>0</mean>
+                          <stddev>0.021</stddev>
+                          <bias_mean>0.05</bias_mean>
+                          <bias_stddev>0.0075</bias_stddev>
+                          <dynamic_bias_stddev>0.000375</dynamic_bias_stddev>
+                          <dynamic_bias_correlation_time>175.0</dynamic_bias_correlation_time>
+                          <precision>0.005</precision>
+                        </noise>
+                      </x>
+                      <y>
+                        <noise type="gaussian">
+                          <mean>0</mean>
+                          <stddev>0.021</stddev>
+                          <bias_mean>0.05</bias_mean>
+                          <bias_stddev>0.0075</bias_stddev>
+                          <dynamic_bias_stddev>0.000375</dynamic_bias_stddev>
+                          <dynamic_bias_correlation_time>175.0</dynamic_bias_correlation_time>
+                          <precision>0.005</precision>
+                        </noise>
+                      </y>
+                      <z>
+                        <noise type="gaussian">
+                          <mean>0</mean>
+                          <stddev>0.021</stddev>
+                          <bias_mean>0.05</bias_mean>
+                          <bias_stddev>0.0075</bias_stddev>
+                          <dynamic_bias_stddev>0.000375</dynamic_bias_stddev>
+                          <dynamic_bias_correlation_time>175.0</dynamic_bias_correlation_time>
+                          <precision>0.005</precision>
+                        </noise>
+                      </z>
+                    </linear_acceleration>
+                  </imu> -->
             </sensor>
         </gazebo>

File: dev_ws/src/diff_robot_description/urdf/sensors/lidar.urdf.xacro (robot description, xacro)
@@ -36,6 +36,6 @@
     enable_collision:=false">
     <xacro:property name="radius" value="${lidar_width/2}" />
-    <xacro:property name="ixx_iyy" value="${(mass/12) * (3 * radius * radius + lidar_height * lidar_height)}" />
-    <xacro:property name="izz" value="${(mass/2) * (radius * radius)}" />
+    <xacro:property name="ixx_iyy" value="1" />
+    <xacro:property name="izz" value="1" />
     <link name="${prefix}${frame_id}">
       <visual>
@@ -71,6 +71,6 @@
       <origin xyz="${xyz_offset}" rpy="${rpy_offset}"/>
     </joint>
-    <!-- Plugin Section for Gazebo-->
-    <gazebo>
+     <!-- Plugin Lidar Sensors Section for Gazebo-->
+     <gazebo>
       <plugin
        filename="gz-sim-sensors-system"

File: dev_ws/src/diff_robot_description/urdf/sensors/rgbd_camera.urdf.xacro (robot description, xacro)
@@ -6,5 +6,4 @@
     camera_name:='cam_1'
     parent:='base_link'
-    mesh_file:='file://$(find yahboom_rosmaster_description)/meshes/intel_realsense/visual/d435.stl'
     xyz_offset:='0.105 0 0.05'
     rpy_offset:='0 -0.50 0'
@@ -36,5 +35,5 @@
     izz:=0.003879257
     material_name:='aluminum'
-    material_color:='0.5 0.5 0.5 1'
+    material_color:='1 0 0 1'
     horizontal_fov:=1.5184
     image_width:=424
@@ -48,7 +47,7 @@
     <link name="${prefix}${camera_name}_link">
       <visual>
-        <origin xyz="${mesh_xyz_offset}" rpy="${mesh_rpy_offset}"/>
+        <origin xyz="0 0 0" rpy="0 0 0"/>
         <geometry>
-          <mesh filename="${mesh_file}" />
+          <box size="${cam_depth} ${cam_width} ${cam_height}"/>
         </geometry>
         <material name="${material_name}">
@@ -58,5 +57,5 @@
       <xacro:if value="${enable_collision}">
         <collision>
-          <origin xyz="${collision_xyz_offset}" rpy="${collision_rpy_offset}"/>
+          <origin xyz="0 0 0" rpy="0 0 0"/>
           <geometry>
             <box size="${cam_depth} ${cam_width} ${cam_height}"/>
